File: iM880B_breakout.sch (KiCad schematic (older format))
At the start: 1 part

Commit message: Whatever
Parts:
- added P1: CONN_01X12, Pin_Headers:Pin_Header_Straight_1x12, symbol CONN_01X12
- added SMA_E1: SMA_EDGE, SMA_EDGE:SMA_EDGE, symbol SMA_EDGE
- U1: renamed from U?; footprint (none) -> iM880B:iM880B
Connections:
- net labels added: P1-IO/JTCK/SWCLK
- wire segments 0 -> 2
Changed lines of the file:
@@
 LIBS:valves
 LIBS:rfcom
+LIBS:sma_edge
+LIBS:iM880B_breakout-cache
 EELAYER 25 0
 EELAYER END
@@
 $EndDescr
 $Comp
-L iM880B U?
+L iM880B U1
 U 1 1 583C5F07
 P 4500 2850
-F 0 "U?" H 4550 3929 50  0000 C CNN
+F 0 "U1" H 4550 3929 50  0000 C CNN
 F 1 "iM880B" H 4550 3837 50  0000 C CNN
-F 2 "" H 4300 1750 50  0000 C CNN
+F 2 "iM880B:iM880B" H 4300 1750 50  0001 C CNN
 F 3 "" H 4300 1750 50  0000 C CNN
 	1    4500 2850
 	1    0    0    -1
 $EndComp
+$Comp
+L SMA_EDGE SMA_E1
+U 1 1 583C9174
+P 6750 4500
+F 0 "SMA_E1" H 7078 4561 60  0000 L CNN
+F 1 "SMA_EDGE" H 7078 4455 60  0000 L CNN
+F 2 "SMA_EDGE:SMA_EDGE" H 6750 4500 60  0001 C CNN
+F 3 "" H 6750 4500 60  0000 C CNN
+	1    6750 4500
+	1    0    0    -1
+$EndComp
+$Comp
+L CONN_01X12 P1
+U 1 1 583C98AA
+P 1550 2500
+F 0 "P1" H 1628 2538 50  0000 L CNN
+F 1 "CONN_01X12" H 1628 2446 50  0000 L CNN
+F 2 "Pin_Headers:Pin_Header_Straight_1x12" H 1550 2500 50  0001 C CNN
+F 3 "" H 1550 2500 50  0000 C CNN
+	1    1550 2500
+	-1   0    0    -1
+$EndComp
+Wire Wire Line
+	1750 1950 2150 1950
+Text Label 1800 1950 0    60   ~ 0
+P1-IO/JTCK/SWCLK
+Wire Wire Line
+	3350 2450 3600 2450
+Text Label 3350 2450 0    60   ~ 0
+P1-IO/JTCK/SWCLK
 $EndSCHEMATC
